Commit message: feat(robot_arm_driver): 驱动栈切换 ros2_canopen(vendored) + 新驱动器真机排坑
自研 CANopenLinux 栈整体下线，替换为 vendored ros2_canopen 0.2.13 精简版；
robot_arm_driver 改容器目录（arm_driver/ 为 ament 包本体 + ros2_canopen/ 兄弟目录）。
real 后端 v2.0：单 controller_manager 管全 6 轴（J1-3 RobotSystem/CANopen +
J4-6 CameraHardwareInterface/HID）。

真机排坑（更换新驱动器后使能/运动失败，逐项总线实测定位）：
- EDS 产品号 0x0006→0x0003：1018 身份校验不匹配导致 master boot 失败
- bus.yml 三关节 boot 下发 6098=0：新驱动出厂回零方法非 0（1/35），402 驱动
  init 强制回零失败导致激活回滚掉使能；绝对编码器标零走 set_encoder_zero
- EDS RPDO3/4 默认值改"禁用"（与实物出厂一致）+ bus.yml 显式启用 RPDO3
  (6040+607A, 立即生效)：否则 dcfgen 认为无差异跳过下发，PP 目标 607A
  帧被驱动器静默丢弃（"能使能不动弹"的根因）
- CAN 口 txqueuelen 须 ≥128（lely CanController 要求，普通用户无权自改，
  EPERM 直接崩栈）：拉起命令文档全量补充
- 云台插件名 emeet_camera_driver→robot_gimbal_driver（云台包改名 URDF 未跟上，
  controller_manager 加载即 abort）
- moveit_controllers_{real,mujoco}.yaml：控制器条目嵌套入
  moveit_simple_controller_manager（顶层写法 action_ns 读取不到）

电机 402 模式切换编排：arm_driver_services v1.1 新增
/arm_node/set_mode_{pp,ip,pv}；controllers_real.yaml arm_controller 改 claim
全 6 轴（跨两硬件组件，命令总线与 Gazebo/MuJoCo 对齐，allow_partial 兼容
visp J1-3 流）+ arm_velocity_controller（PV 备用，--inactive 预加载）；
real.launch 按 controller 自动选模式（joint_position→PP，轨迹类→IP 默认，
PV 待 servo/visp 上层改发速度指令后接入）。

真机验证：三轴 boot+使能、PP 0→0.2rad→0（跟踪~15counts）、
IP 0.045→0.15rad 匀速平滑跟随、回零精确，全部通过。

Co-Authored-By: Claude Fable 5 <noreply@anthropic.com>
Change-Id: I58d2c6360578fab1b248b81ecc41facb97c6b006

File: robot_arm_description/urdf/arm.urdf.xacro (robot description, xacro)
@@ -49,4 +49,5 @@
                      backend:='gazebo'
                      arm_sim_mode:='false'
+                     can_interface:='can0'
                      emit_camera_control:='true'
                      controllers_yaml:=''">
@@ -186,5 +187,5 @@
     <child link="Link1"/>
     <axis xyz="0 0 1"/>
-    <limit lower="-3.1" upper="3.1" effort="5" velocity="3.14"/>
+    <limit lower="-2.618" upper="2.618" effort="5" velocity="3.14"/>
     <dynamics damping="1.0" friction="0.0"/>
   </joint>
@@ -242,15 +243,21 @@
        Arm joints 1-3：
          backend=gazebo（默认）→ GazeboSystem（Gazebo 仿真）
-         backend=real          → robot_arm_driver/ArmHardwareInterface（CANopen 实物）
-                                 arm_sim_mode=true 时仅回显命令、不连 CAN（干跑）
+         backend=real          → canopen_ros2_control/RobotSystem（ros2_canopen，CiA402 实物）
+                                 总线拓扑/换算/PDO 见 robot_arm_driver/config/canopen/bus.yml
+                                 arm_sim_mode=true → mock_components/GenericSystem
+                                                     （命令回显为状态，不连 CAN，干跑）
        ═══════════════════════════════════════════════════════════════════════ -->
   <ros2_control name="eMeetArm_hardware" type="system">
     <hardware>
       <xacro:if value="${backend == 'real'}">
-        <plugin>robot_arm_driver/ArmHardwareInterface</plugin>
-        <!-- 硬件参数（CAN/node_id/编码器分辨率等）在此 yaml 里改，无需动 xacro -->
-        <param name="config_file">$(find robot_arm_driver)/config/arm_hw.yaml</param>
-        <xacro:if value="${arm_sim_mode}"><param name="sim_mode">true</param></xacro:if>
-        <xacro:unless value="${arm_sim_mode}"><param name="sim_mode">false</param></xacro:unless>
+        <xacro:unless value="${arm_sim_mode}">
+          <plugin>canopen_ros2_control/RobotSystem</plugin>
+          <param name="bus_config">$(find robot_arm_driver)/config/canopen/bus.yml</param>
+          <param name="master_config">$(find robot_arm_driver)/config/canopen/master.dcf</param>
+          <param name="can_interface_name">${can_interface}</param>
+        </xacro:unless>
+        <xacro:if value="${arm_sim_mode}">
+          <plugin>mock_components/GenericSystem</plugin>
+        </xacro:if>
       </xacro:if>
       <xacro:unless value="${backend == 'real'}">
@@ -259,7 +266,8 @@
     </hardware>
     <joint name="Joint1">
-      <command_interface name="position">
-        <param name="min">-3.1</param>
-        <param name="max">3.1</param>
+      <param name="device_name">joint_1</param>
+      <command_interface name="position">
+        <param name="min">-2.618</param>
+        <param name="max">2.618</param>
       </command_interface>
       <command_interface name="velocity"/>
@@ -268,4 +276,5 @@
     </joint>
     <joint name="Joint2">
+      <param name="device_name">joint_2</param>
       <command_interface name="position">
         <param name="min">-0.8</param>
@@ -277,4 +286,5 @@
     </joint>
     <joint name="Joint3">
+      <param name="device_name">joint_3</param>
       <command_interface name="position">
         <param name="min">-3.14</param>
@@ -300,5 +310,5 @@
       </xacro:if>
       <xacro:unless value="${gazebo_camera}">
-        <plugin>emeet_camera_driver/CameraHardwareInterface</plugin>
+        <plugin>robot_gimbal_driver/CameraHardwareInterface</plugin>
         <param name="camera_type">auto</param>
         <xacro:if value="${sim_mode}">

File: robot_arm_description/urdf/arm_sim.urdf.xacro (robot description, xacro)
@@ -19,4 +19,5 @@
   <xacro:arg name="backend"             default="gazebo"/>
   <xacro:arg name="arm_sim_mode"        default="false"/>
+  <xacro:arg name="can_interface"       default="can0"/>
   <xacro:arg name="emit_camera_control" default="true"/>
   <xacro:arg name="controllers_yaml"    default=""/>
@@ -31,4 +32,5 @@
       backend="$(arg backend)"
       arm_sim_mode="$(arg arm_sim_mode)"
+      can_interface="$(arg can_interface)"
       emit_camera_control="$(arg emit_camera_control)"
       controllers_yaml="$(arg controllers_yaml)"/>

File: robot_arm_description/urdf/eMeetArm_models.urdf (robot description, URDF)
Before this commit: robot eMeetArm_models, 10 links, 9 joints
Joints:
- joint Joint1: limit lower=-3.1 upper=3.1 effort=5 velocity=3.14 -> lower=-2.618 upper=2.618 effort=5 velocity=3.14
