Commit message: feat(mode): 力矩模式 JOINT_EFFORT 在仿真开通，含 pinocchio 重力补偿
ModeManager 的力矩脚手架（参数/总线/看门狗/拒绝逻辑）、bus.yml 的
effort_mode:4(PT)、cia402_data 的 HW_IF_EFFORT 导出本来就在，本次把缺的几环接上：

- URDF：J1-3 加 effort 命令接口（min/max 取 <limit effort>：5/30/5 N·m）。
  effort **状态**接口只给非 real 后端 —— RobotSystem 的 read_state() 不读转矩、
  TPDO 也没映 6077，实物声明了拿不到值，反而会让 jsb 找不到接口。
- controllers.yaml：新增 arm_effort_controller（JointGroupEffortController，只 claim J1-3）；
  gazebo.launch.py 以 --inactive 加载并给 mode_manager 传 effort_controller。
  real.launch.py 故意不配 —— 留空 = 切 JOINT_EFFORT 被明确拒绝，这是安全默认。
- launch_common.mode_manager_node() 增 effort_controller 形参。
- JointLimit 加 effort 字段（从 URDF 解析），力矩限幅用它，不写死常量。
- GUI 新增「力矩控制」页：切模式 + 三轴按住即施力 + 实际力矩回读。

重力补偿（新增 motion/GravityModel，pinocchio）——力矩模式可用的前提：

零指令力矩不是"停住"而是**自由下垂**：实测切进力矩模式后 J2 立刻从 +0.500 砸到
下限 -0.981、J3 从 -1.000 砸到上限 +0.020。故力矩通路改为定时节拍（默认 100Hz），
下发 = g(q) + 用户增量 − d·q̇，再限幅 + 限位刹车。连带三条：
  ① 用户指令只是"重力之上的增量"，存起来由节拍消费，不直接下发；
  ② publishZero() 对力矩模式只清用户增量、不发字面 0，急停/断流同理
     （力矩模式下"停住"就是继续托住）；
  ③ 必须持续发 —— ForwardCommandController 会一直把最后一帧写给硬件，
     位形一变那帧重力力矩就不再平衡。
GravityModel::gravity() 是 fail-closed：位形不全就整体放弃，用默认值顶替缺失
关节会算出错误的**主动力**，比不补偿危险得多。惯量仍以 URDF 为单一真相源。

阻尼项 effort_damping（默认 1.5 N·m·s/rad）：纯重力补偿无耗散，残差会积分成
漂移 —— 实测无阻尼 8s 内 J2 上飘 0.100 rad，加阻尼降到 0.081，松手滑行从
+0.12 降到 +0.05。

Gazebo 实测：切入/切回可重复；gimbal_controller 随主切换自动顶住 J4-6；
限幅（发 999 N·m → 输出 5.0）、长度校验、模式闸（非力矩模式发力矩 → 丢弃）均生效；
悬停 8s 漂移 J2 0.081 / J3 0.032 rad；J1 施 +0.5 N·m 只有 J1 动（耦合已补掉）；
切回轨迹模式后位置精确回到 J2=+0.5000 J3=-1.0000。

仿真里仍有约 0.01 rad/s 单向漂移（Gazebo 关节无摩擦，真机谐波减速器摩擦大得多），
要彻底锁住得加位置弹簧项 —— 那已经是阻抗控制（P3 的 ADMITTANCE），未做。

实物未开通，缺两件：① 6071 单位是「0.1% 额定转矩」而本层是 N·m，换算系数要查
手册额定转矩（vendored ros2_canopen 的 scale_eff_* 上游未实现，按 VENDOR.md
不改 vendored，换算应落在 relay 层）；② 6077 力矩反馈没映进 TPDO
（TPDO1 还空 5 字节，6077 是 INTEGER16 只占 2B）。

新增依赖：pinocchio（robot_arm_node 此前没有任何动力学库）。

Change-Id: Ic8331cfcba56f8c3d979486bd6856ce46a503aba

File: robot_arm_description/urdf/arm.urdf.xacro (robot description, xacro)
@@ -245,6 +245,21 @@
       </command_interface>
       <command_interface name="velocity"/>
+      <!-- JOINT_EFFORT 模式（2026-08-11 开通）：min/max 取 <limit effort>，单位 N·m。
+           实物侧 bus.yml 已配 effort_mode:4(PT)，cia402_data 见到本接口才会 export
+           HW_IF_EFFORT → set_target 写 6071；仿真侧 GazeboSystem 直接 SetForce。
+           同关节的 position/velocity/effort 三个命令接口互斥，同一时刻只准一个
+           控制器 claim（由 mode_manager_node 经 switch_controller 仲裁）。 -->
+      <command_interface name="effort">
+        <param name="min">-5.0</param>
+        <param name="max">5.0</param>
+      </command_interface>
       <state_interface name="position"><param name="initial_value">0.0</param></state_interface>
       <state_interface name="velocity"/>
+      <!-- 力矩回读只在仿真侧声明：RobotSystem 的 read_state() 不读转矩（TPDO 也没映
+           6077），实物声明了也拿不到值，反而会让 joint_state_broadcaster 找不到接口。
+           实物要力矩反馈得先把 6077 映进 TPDO1（那里还空 5 字节）。 -->
+      <xacro:unless value="${backend == 'real'}">
+        <state_interface name="effort"/>
+      </xacro:unless>
     </joint>
     <joint name="Joint2">
@@ -272,6 +287,14 @@
       </command_interface>
       <command_interface name="velocity"/>
+      <!-- J2 扛整臂重力，<limit effort> 是 30 N·m（三轴里最大）。见 Joint1 注释。 -->
+      <command_interface name="effort">
+        <param name="min">-30.0</param>
+        <param name="max">30.0</param>
+      </command_interface>
       <state_interface name="position"><param name="initial_value">0.0</param></state_interface>
       <state_interface name="velocity"/>
+      <xacro:unless value="${backend == 'real'}">
+        <state_interface name="effort"/>
+      </xacro:unless>
     </joint>
     <joint name="Joint3">
@@ -299,6 +322,14 @@
       </command_interface>
       <command_interface name="velocity"/>
+      <!-- 见 Joint1 注释；<limit effort> 5 N·m。 -->
+      <command_interface name="effort">
+        <param name="min">-5.0</param>
+        <param name="max">5.0</param>
+      </command_interface>
       <state_interface name="position"><param name="initial_value">0.0</param></state_interface>
       <state_interface name="velocity"/>
+      <xacro:unless value="${backend == 'real'}">
+        <state_interface name="effort"/>
+      </xacro:unless>
     </joint>
   </ros2_control>
